File: hardware/breakneck/breakneck.kicad_pcb (KiCad board)
At the start: 2 copper layers, 53.3 x 64 mm, 124 parts, among them J1 CONN_WEST, J10 GS2, J12 CONN_JTAG_6P, J15 GS2, J16 CONN_JST, J2 CONN_DEDI, J3 CONN_OLED, J4 USB_C_Rcpt_Min, J5 CONN_SOUTH, J6 CONN_EAST, J8 CONN_JTAG_TC, SW1 SW_SPST, SW2 SW_SPST, SW3 SW_SPST, SW4 SW_SPDT, U1 ATECC508A, U2 SST26VF064B, U3 CEC1702, U4 CP2102N, U5 MIC5377YC5, U6 LN6206P33M, U7 LN6206P15M, X1 Badgelife_shitty, Y1 Crystal

Commit message: master
Parts:
- BT1: footprint Monero_Local:Keystone_3000_1x12mm-CoinCell -> ByteRub_Local:Keystone_3000_1x12mm-CoinCell
- C1, C10, C11, C12, C13, C14, C15, C18, C19, C2, C21, C22, C23, C24, C25, C26, C27, C28, C29, C3, C30, C31, C32, C4, C5, C6, C7, C8, C9: footprint Monero_Local:C_0805 -> ByteRub_Local:C_0805
- D+, D-, TP1, TP10, TP12, TP13, TP14, TP15, TP18, TP2, TP21, TP22, TP5, TP6, VOTP: footprint Monero_Local:TestPoint_THTPad_D1.5mm_Drill0.7mm -> ByteRub_Local:TestPoint_THTPad_D1.5mm_Drill0.7mm
- D1, U6, U7: footprint Monero_Local:SOT-23 -> ByteRub_Local:SOT-23
- D2: footprint Monero_Local:SOT-143 -> ByteRub_Local:SOT-143
- D5: footprint Monero_Local:D_SOD-123 -> ByteRub_Local:D_SOD-123
- D6, D7, RX, TX: footprint Monero_Local:LED_0805 -> ByteRub_Local:LED_0805
- DS1: footprint Monero_Local:Eastrising_ER-CON30HT-1_01x30_P0.50mm -> ByteRub_Local:Eastrising_ER-CON30HT-1_01x30_P0.50mm
- FID1, FID2, FID3, FID4, FID5, FID6: footprint Monero_Local:Fiducial_1mm_Dia_2.54mm_Outer_CopperTop -> ByteRub_Local:Fiducial_1mm_Dia_2.54mm_Outer_CopperTop
- J1, J6: footprint Monero_Local:Pin_Header_Straight_1x20_Pitch2.54mm -> ByteRub_Local:Pin_Header_Straight_1x20_Pitch2.54mm
- J10, J15, OTP, R1, R10, R11, R12, R13, R15, R16, R17, R18, R19, R2, R20, R21, R22, R23, R24, R25, R26, R27, R28, R29, R3, R4, R5, R6, R7, R8, R9: footprint Monero_Local:R_0805 -> ByteRub_Local:R_0805
- J12: footprint Monero_Local:PinSocket_2x05_P2.54mm_Vertical -> ByteRub_Local:PinSocket_2x05_P2.54mm_Vertical
- J16: footprint Monero_Local:JST_PH_B2B-PH-K_02x2.00mm_Straight -> ByteRub_Local:JST_PH_B2B-PH-K_02x2.00mm_Straight
- J2: footprint Monero_Local:Pin_Header_Straight_2x04_Pitch2.54mm -> ByteRub_Local:Pin_Header_Straight_2x04_Pitch2.54mm
- J3: footprint Monero_Local:Socket_Strip_Straight_1x07_Pitch2.54mm -> ByteRub_Local:Socket_Strip_Straight_1x07_Pitch2.54mm
- J4: footprint Monero_Local:USBC_Rcpt_Min_12401610E4-2A -> ByteRub_Local:USBC_Rcpt_Min_12401610E4-2A
- J5: footprint Monero_Local:Pin_Header_Straight_1x14_Pitch2.54mm -> ByteRub_Local:Pin_Header_Straight_1x14_Pitch2.54mm
- J8: footprint Monero_Local:Tag-Connect_TC2050-IDC-NL -> ByteRub_Local:Tag-Connect_TC2050-IDC-NL
- JCC, JDM, JDP: footprint Monero_Local:Solderjump-2NCRndpad -> ByteRub_Local:Solderjump-2NCRndpad
- JP1, JP2: footprint Monero_Local:Pin_Header_Angled_1x02_Pitch2.54mm -> ByteRub_Local:Pin_Header_Angled_1x02_Pitch2.54mm
- LOGO1: value Monerologo-mid -> ByteRublogo-mid; footprint Monero_Local:MoneroCircleCombi -> ByteRub_Local:ByteRubCircleCombi
- LOGOTXT1: value Monerologo-txt -> ByteRublogo-txt; footprint MoneroTextSilk -> ByteRubTextSilk
- MH1, MH2, MH3: footprint Monero_Local:MountingHole_3mm_Pad_Via -> ByteRub_Local:MountingHole_3mm_Pad_Via
- SW1, SW2: footprint Monero_Local:SW_SPST_K21102SP -> ByteRub_Local:SW_SPST_K21102SP
- SW3: footprint Monero_Local:SW_SPST_ESE11MV1 -> ByteRub_Local:SW_SPST_ESE11MV1
- SW4: footprint Monero_Local:SW_SPDT_CLSB-12A -> ByteRub_Local:SW_SPDT_CLSB-12A
- TP26, TP27: footprint Monero_Local:TestPoint_THTPad_1.0x1.0mm_Drill0.5mm -> ByteRub_Local:TestPoint_THTPad_1.0x1.0mm_Drill0.5mm
- U1: footprint Monero_Local:DFN-8-1EP_2x3mm_Pitch0.5mm -> ByteRub_Local:DFN-8-1EP_2x3mm_Pitch0.5mm
- U2: footprint Monero_Local:DFN-S-8-1EP_6x5mm_Pitch1.27mm -> ByteRub_Local:DFN-S-8-1EP_6x5mm_Pitch1.27mm
- U3: footprint Monero_Local:WFBGACEC1702 -> ByteRub_Local:WFBGACEC1702
- U4: footprint Monero_Local:QFN-28-1EP_5x5mm_Pitch0.5mm -> ByteRub_Local:QFN-28-1EP_5x5mm_Pitch0.5mm
- U5: footprint Monero_Local:SOT-353_SC-70-5 -> ByteRub_Local:SOT-353_SC-70-5
- X1: footprint Monero_Local:Badgelife-Shitty-2x2 -> ByteRub_Local:Badgelife-Shitty-2x2
- Y1: footprint Monero_Local:Crystal_SMD_3215-2Pin_3.2x1.5mm -> ByteRub_Local:Crystal_SMD_3215-2Pin_3.2x1.5mm
Other:
- board text added: "Seventh generation prototype RFC-HWALLET-1 ET1 Extra Tabulo, by the ByteRub Hardware Team CERN OSH License, © 2019 The ByteRub Project"
- board text removed: "Seventh generation prototype RFC-HWALLET-1 ET1 Extra Tabulo, by the Monero Hardware Team CERN OSH License, © 2019 The Monero Project"
