File: hardware/breakneck/breakpanel.kicad_pcb (KiCad board)
At the start: 2 copper layers, 145 x 165 mm, 690 parts, among them J1 CONN_WEST, J10 GS2, J12 CONN_JTAG_6P, J15 GS2, J16 CONN_JST, J2 CONN_DEDI, J3 CONN_OLED, J4 USB_C_Receptacle, J5 CONN_SOUTH, J6 CONN_EAST, J8 CONN_JTAG_TC, SW1 SW_SPST, SW2 SW_SPST, U1 ATECC508A, U2 SST26VF064B, U3 CEC1702, U4 CP2102N, U6 LN6206P33M, U7 LN6206P15M, X1 Badgelife_shitty, Y1 Crystal

Commit message: master
Parts:
- BT1 (x6): footprint Monero_Local:Keystone_3000_1x12mm-CoinCell -> ByteRub_Local:Keystone_3000_1x12mm-CoinCell
- C1 (x6), C10 (x6), C11 (x6), C12 (x6), C13 (x6), C14 (x6), C15 (x6), C18 (x6), C19 (x6), C2 (x6), C21 (x6), C22 (x6), C23 (x6), C26 (x6), C28 (x6), C29 (x6), C3 (x6), C30 (x6), C31 (x6), C32 (x6), C4 (x6), C5 (x6), C6 (x6), C7 (x6), C8 (x6), C9 (x6): footprint Monero_Local:C_0805 -> ByteRub_Local:C_0805
- D1 (x6), U6 (x6), U7 (x6): footprint Monero_Local:SOT-23 -> ByteRub_Local:SOT-23
- D2 (x6): footprint Monero_Local:SOT-143 -> ByteRub_Local:SOT-143
- D5 (x6): footprint Monero_Local:D_SOD-123 -> ByteRub_Local:D_SOD-123
- D6 (x6), D7 (x6), RX (x6), TX (x6): footprint Monero_Local:LED_0805 -> ByteRub_Local:LED_0805
- DS1 (x6): footprint Monero_Local:Eastrising_ER-CON30HT-1_01x30_P0.50mm -> ByteRub_Local:Eastrising_ER-CON30HT-1_01x30_P0.50mm
- FID1 (x6), FID2 (x6), FID3 (x6), FID4 (x6), FID5 (x6), FID6 (x6): footprint Monero_Local:Fiducial_1mm_Dia_2.54mm_Outer_CopperTop -> ByteRub_Local:Fiducial_1mm_Dia_2.54mm_Outer_CopperTop
- J1 (x6), J6 (x6): footprint Monero_Local:Pin_Header_Straight_1x20_Pitch2.54mm -> ByteRub_Local:Pin_Header_Straight_1x20_Pitch2.54mm
- J10 (x6), J15 (x6), OTP (x6), R1 (x6), R10 (x6), R11 (x6), R12 (x6), R13 (x6), R15 (x6), R16 (x6), R17 (x6), R18 (x6), R19 (x6), R2 (x6), R20 (x6), R21 (x6), R25 (x6), R26 (x6), R27 (x6), R28 (x6), R3 (x6), R4 (x6), R5 (x6), R6 (x6), R7 (x6), R8 (x6), R9 (x6): footprint Monero_Local:R_0805 -> ByteRub_Local:R_0805
- J12 (x6): footprint Monero_Local:PinSocket_2x05_P2.54mm_Vertical -> ByteRub_Local:PinSocket_2x05_P2.54mm_Vertical
- J16 (x6): footprint Monero_Local:JST_PH_B2B-PH-K_02x2.00mm_Straight -> ByteRub_Local:JST_PH_B2B-PH-K_02x2.00mm_Straight
- J2 (x6): footprint Monero_Local:Pin_Header_Straight_2x04_Pitch2.54mm -> ByteRub_Local:Pin_Header_Straight_2x04_Pitch2.54mm
- J3 (x6): footprint Monero_Local:Socket_Strip_Straight_1x07_Pitch2.54mm -> ByteRub_Local:Socket_Strip_Straight_1x07_Pitch2.54mm
- J4 (x6): footprint Monero_Local:USB_C_Receptacle_Amphenol_12401610E4-2A -> ByteRub_Local:USB_C_Receptacle_Amphenol_12401610E4-2A
- J5 (x6): footprint Monero_Local:Pin_Header_Straight_1x14_Pitch2.54mm -> ByteRub_Local:Pin_Header_Straight_1x14_Pitch2.54mm
- J8 (x6): footprint Monero_Local:Tag-Connect_TC2050-IDC-NL -> ByteRub_Local:Tag-Connect_TC2050-IDC-NL
- JP1 (x6), JP2 (x6): footprint Monero_Local:Pin_Header_Angled_1x02_Pitch2.54mm -> ByteRub_Local:Pin_Header_Angled_1x02_Pitch2.54mm
- LOGO1 (x6): value Monerologo-mid -> ByteRublogo-mid; footprint Monero_Local:MoneroCircleCombi -> ByteRub_Local:ByteRubCircleCombi
- LOGOTXT1 (x6): value Monerologo-txt -> ByteRublogo-txt; footprint MoneroTextSilk -> ByteRubTextSilk
- MH1 (x6), MH2 (x6), MH3 (x6): footprint Monero_Local:MountingHole_3mm_Pad_Via -> ByteRub_Local:MountingHole_3mm_Pad_Via
- SW1 (x6), SW2 (x6): footprint Monero_Local:SW_SPST_K21102SP -> ByteRub_Local:SW_SPST_K21102SP
- TAB1, TAB11, TAB12, TAB15, TAB16, TAB2, TAB21, TAB22, TAB25, TAB26, TAB5, TAB6: footprint Monero_HW:Panel_Mousetab_25mm_Single -> ByteRub_HW:Panel_Mousetab_25mm_Single
- TAB10, TAB13, TAB14, TAB17, TAB18, TAB19, TAB20, TAB23, TAB24, TAB3, TAB4, TAB7, TAB8, TAB9: footprint Monero_Local:Panel_Mousetab_25mm_Double -> ByteRub_Local:Panel_Mousetab_25mm_Double
- TP1 (x6), TP10 (x6), TP12 (x6), TP13 (x6), TP14 (x6), TP15 (x6), TP18 (x6), TP19 (x6), TP2 (x6), TP20 (x6), TP21 (x6), TP22 (x6), TP5 (x6), TP6 (x6), VOTP (x6): footprint Monero_Local:TestPoint_THTPad_D1.5mm_Drill0.7mm -> ByteRub_Local:TestPoint_THTPad_D1.5mm_Drill0.7mm
- U1 (x6): footprint Monero_Local:DFN-8-1EP_2x3mm_Pitch0.5mm -> ByteRub_Local:DFN-8-1EP_2x3mm_Pitch0.5mm
- U2 (x6): footprint Monero_Local:DFN-S-8-1EP_6x5mm_Pitch1.27mm -> ByteRub_Local:DFN-S-8-1EP_6x5mm_Pitch1.27mm
- U3 (x6): footprint Monero_Local:WFBGACEC1702 -> ByteRub_Local:WFBGACEC1702
- U4 (x6): footprint Monero_Local:QFN-28-1EP_5x5mm_Pitch0.5mm -> ByteRub_Local:QFN-28-1EP_5x5mm_Pitch0.5mm
- X1 (x6): footprint Monero_Local:Badgelife-Shitty-2x2 -> ByteRub_Local:Badgelife-Shitty-2x2
- Y1 (x6): footprint Monero_Local:Crystal_SMD_3215-2Pin_3.2x1.5mm -> ByteRub_Local:Crystal_SMD_3215-2Pin_3.2x1.5mm
Other:
- board text added: "Panelised by the ByteRub Hardware team, January 2019"
- board text added: "Seventh generation prototype RFC-HWALLET-1 ET1 Extra Tabulo, by the ByteRub Hardware Team CERN OSH License, © 2019 The ByteRub Project"
- board text added: "Stencil8 calibrated, write ByteRub Hardware for details"
- board text removed: "Panelised by the Monero Hardware team, January 2019"
- board text removed: "Seventh generation prototype RFC-HWALLET-1 ET1 Extra Tabulo, by the Monero Hardware Team CERN OSH License, © 2019 The Monero Project"
- board text removed: "Stencil8 calibrated, write Monero Hardware for details"
