File: hardware/breaknext/breaknext.kicad_pcb (KiCad board)
At the start: 2 copper layers, 53.3 x 64 mm, 15 parts

Commit message: master
Parts:
- FID3, REF**: footprint Monero_Local:Fiducial_1mm_Dia_2.54mm_Outer_CopperBottom -> ByteRub_Local:Fiducial_1mm_Dia_2.54mm_Outer_CopperBottom
- LOGO1: value Monerologo-mid -> ByteRublogo-mid; footprint Monero_Local:MoneroCircleCombi -> ByteRub_Local:ByteRubCircleCombi
- REF** (x3): footprint Monero_Local:MountingHole_3mm_Pad_Via -> ByteRub_Local:MountingHole_3mm_Pad_Via
- REF** (x2): footprint Monero_Local:Socket_Strip_Straight_1x20_Pitch2.54mm -> ByteRub_Local:Socket_Strip_Straight_1x20_Pitch2.54mm
- REF**: footprint Monero_Local:Socket_Strip_Straight_1x14_Pitch2.54mm -> ByteRub_Local:Socket_Strip_Straight_1x14_Pitch2.54mm
- REF**: footprint Monero_Local:JST_PH_B2B-PH-K_02x2.00mm_Straight -> ByteRub_Local:JST_PH_B2B-PH-K_02x2.00mm_Straight
- REF**: footprint Monero_Local:microSD_Card_Receptacle_Hirose_DM3AT-SF-PEJM5 -> ByteRub_Local:microSD_Card_Receptacle_Hirose_DM3AT-SF-PEJM5
- REF** (x4): footprint Monero_Local:Fiducial_1mm_Dia_2.54mm_Outer_CopperTop -> ByteRub_Local:Fiducial_1mm_Dia_2.54mm_Outer_CopperTop
Changed lines of the file:
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@@
     (date 2018-01-10)
     (rev 0.7.5)
-    (company "The Monero Project, Hardware Team")
-    (comment 1 "Copyright © 2018, The Monero Project")
+    (company "The ByteRub Project, Hardware Team")
+    (comment 1 "Copyright © 2018, The ByteRub Project")
     (comment 2 "Fulfilling the developer edition role")
     (comment 3 "Pending quality assurance testing")
@@
     (add_net "Net-(J6-Pad1)")
   )
-  (module Monero_Local:MountingHole_3mm_Pad_Via (layer F.Cu)
+  (module ByteRub_Local:MountingHole_3mm_Pad_Via (layer F.Cu)
     (at 145.72 67.04)
     (descr "Mounting Hole 3mm")
@@
       (net 1 GND))
   )
-  (module Monero_Local:MountingHole_3mm_Pad_Via (layer F.Cu)
+  (module ByteRub_Local:MountingHole_3mm_Pad_Via (layer F.Cu)
     (at 107.62 67.04)
     (descr "Mounting Hole 3mm")
@@
       (net 1 GND))
   )
-  (module Monero_Local:MountingHole_3mm_Pad_Via (layer F.Cu)
+  (module ByteRub_Local:MountingHole_3mm_Pad_Via (layer F.Cu)
     (at 125.4 117.84)
     (descr "Mounting Hole 3mm")
@@
       (net 1 GND))
   )
-  (module Monero_Local:Fiducial_1mm_Dia_2.54mm_Outer_CopperTop (layer F.Cu)
+  (module ByteRub_Local:Fiducial_1mm_Dia_2.54mm_Outer_CopperTop (layer F.Cu)
     (at 102 66)
     (descr "Circular Fiducial, 1mm bare copper top; 2.54mm keepout")
@@
       (net 7 "Net-(FID1-Pad~)") (solder_mask_margin 0.77) (clearance 0.77))
   )
-  (module Monero_Local:Fiducial_1mm_Dia_2.54mm_Outer_CopperTop (layer F.Cu)
+  (module ByteRub_Local:Fiducial_1mm_Dia_2.54mm_Outer_CopperTop (layer F.Cu)
     (at 151.34 126)
     (descr "Circular Fiducial, 1mm bare copper top; 2.54mm keepout")
@@
       (net 8 "Net-(FID2-Pad~)") (solder_mask_margin 0.77) (clearance 0.77))
   )
-  (module Monero_Local:Fiducial_1mm_Dia_2.54mm_Outer_CopperBottom (layer F.Cu)
+  (module ByteRub_Local:Fiducial_1mm_Dia_2.54mm_Outer_CopperBottom (layer F.Cu)
     (at 102 66)
     (descr "Circular Fiducial, 1mm bare copper bottom; 2.54mm keepout")
@@
       (net 9 "Net-(FID3-Pad~)") (solder_mask_margin 0.77) (clearance 0.77))
   )
-  (module Monero_Local:Fiducial_1mm_Dia_2.54mm_Outer_CopperBottom (layer F.Cu)
+  (module ByteRub_Local:Fiducial_1mm_Dia_2.54mm_Outer_CopperBottom (layer F.Cu)
     (at 151.34 126)
     (descr "Circular Fiducial, 1mm bare copper bottom; 2.54mm keepout")
@@
       (net 10 "Net-(FID4-Pad~)") (solder_mask_margin 0.77) (clearance 0.77))
   )
-  (module Monero_Local:MoneroCircleCombi (layer B.Cu)
+  (module ByteRub_Local:ByteRubCircleCombi (layer B.Cu)
     (at 143.25 78 180)
     (fp_text reference LOGO1 (at 0 0 180) (layer B.SilkS) hide
       (effects (font (thickness 0.3)) (justify mirror))
     )
-    (fp_text value Monerologo-mid (at 0.75 0 180) (layer B.SilkS) hide
+    (fp_text value ByteRublogo-mid (at 0.75 0 180) (layer B.SilkS) hide
       (effects (font (thickness 0.3)) (justify mirror))
     )
@@
       (xy -2.187393 5.584652) (xy -1.270442 5.872224) (xy -0.340435 6.012336) (xy 0.587929 6.006769)) (layer B.Mask) (width 0.01))
   )
-  (module Monero_Local:Fiducial_1mm_Dia_2.54mm_Outer_CopperTop (layer B.Cu)
+  (module ByteRub_Local:Fiducial_1mm_Dia_2.54mm_Outer_CopperTop (layer B.Cu)
     (at 151.34 66)
     (descr "Circular Fiducial, 1mm bare copper top; 2.54mm keepout")
@@
       (solder_mask_margin 0.77) (clearance 0.77))
   )
-  (module Monero_Local:Fiducial_1mm_Dia_2.54mm_Outer_CopperTop (layer F.Cu)
+  (module ByteRub_Local:Fiducial_1mm_Dia_2.54mm_Outer_CopperTop (layer F.Cu)
     (at 151.34 66)
     (descr "Circular Fiducial, 1mm bare copper top; 2.54mm keepout")
@@
       (solder_mask_margin 0.77) (clearance 0.77))
   )
-  (module Monero_Local:Socket_Strip_Straight_1x20_Pitch2.54mm (layer F.Cu)
+  (module ByteRub_Local:Socket_Strip_Straight_1x20_Pitch2.54mm (layer F.Cu)
     (at 102.54 120.38 180)
     (descr "Through hole straight socket strip, 1x20, 2.54mm pitch, single row")
@@
     )
   )
-  (module Monero_Local:Socket_Strip_Straight_1x20_Pitch2.54mm (layer F.Cu)
+  (module ByteRub_Local:Socket_Strip_Straight_1x20_Pitch2.54mm (layer F.Cu)
     (at 150.8 120.38 180)
     (descr "Through hole straight socket strip, 1x20, 2.54mm pitch, single row")
@@
     )
   )
-  (module Monero_Local:Socket_Strip_Straight_1x14_Pitch2.54mm (layer F.Cu)
+  (module ByteRub_Local:Socket_Strip_Straight_1x14_Pitch2.54mm (layer F.Cu)
     (at 102.54 125.46 90)
     (descr "Through hole straight socket strip, 1x14, 2.54mm pitch, single row")
@@
     )
   )
-  (module Monero_Local:JST_PH_B2B-PH-K_02x2.00mm_Straight (layer F.Cu)
+  (module ByteRub_Local:JST_PH_B2B-PH-K_02x2.00mm_Straight (layer F.Cu)
     (at 133.25 120.5)
     (descr "JST PH series connector, B2B-PH-K, top entry type, through hole, Datasheet: http://www.jst-mfg.com/product/pdf/eng/ePH.pdf")
@@
     )
   )
-  (module Monero_Local:microSD_Card_Receptacle_Hirose_DM3AT-SF-PEJM5 (layer F.Cu)
+  (module ByteRub_Local:microSD_Card_Receptacle_Hirose_DM3AT-SF-PEJM5 (layer F.Cu)
     (at 113.5 112)
     (descr "MicroSD card socket")
