File: hardware/confbadge/hcppnfc/hcppnfc.kicad_pcb (KiCad board)
At the start: 2 copper layers, 80 x 71 mm, 13 parts, among them SW1 SW_SPST, SW2 SW_SPST, U1 M24SR02-YMN, U2 M24SR02-YMN

Commit message: master
Parts:
- AE1: footprint Monero_HW:NFCAntennatall -> ByteRub_HW:NFCAntennatall
- FID1, FID2, FID3: footprint Monero_HW:Fiducial_1mm_Dia_2mm_Outer -> ByteRub_HW:Fiducial_1mm_Dia_2mm_Outer
- GFX*: footprint Monero_HW:HCPPNewordtri -> ByteRub_HW:HCPPNewordtri
- GFX*: footprint Monero_HW:HCPPNewordconf -> ByteRub_HW:HCPPNewordconf
- GFX*: footprint Monero_HW:HCPPNewordinst -> ByteRub_HW:HCPPNewordinst
- LOGO*: footprint Monero_HW:HCPPSponsors -> ByteRub_HW:HCPPSponsors
- MH1: footprint Monero_HW:MountingHole_4.3mm_M4_ISO14580_Pad -> ByteRub_HW:MountingHole_4.3mm_M4_ISO14580_Pad
- SW1: footprint Monero_HW:SW_SPST_K21102SP -> ByteRub_HW:SW_SPST_K21102SP
- SW2: footprint Monero_HW:SW_SPST_PTS645 -> ByteRub_HW:SW_SPST_PTS645
- U1, U2: footprint Monero_HW:SOIC-8_3.9x4.9mm_Pitch1.27mm -> ByteRub_HW:SOIC-8_3.9x4.9mm_Pitch1.27mm
Changed lines of the file:
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@@
     (date 2019-04-16)
     (rev 0.8.1)
-    (company "The Monero Project, Hardware Team")
-    (comment 1 "Copyright © 2019, The Monero Project")
+    (company "The ByteRub Project, Hardware Team")
+    (comment 1 "Copyright © 2019, The ByteRub Project")
     (comment 2 "Fulfilling the fourth annual conference badge")
     (comment 3 "Pending quality assurance testing")
@@
     (add_net VCC)
   )
-  (module Monero_HW:HCPPNewordtri (layer F.Cu)
+  (module ByteRub_HW:HCPPNewordtri (layer F.Cu)
     (at 140 90)
     (fp_text reference GFX* (at 0 0) (layer F.SilkS) hide
@@
       (xy 12.671778 19.120556)) (layer F.SilkS) (width 0.01))
   )
-  (module Monero_HW:NFCAntennatall (layer B.Cu)
+  (module ByteRub_HW:NFCAntennatall (layer B.Cu)
     (at 140 93 180)
     (fp_text reference AE1 (at 0 1 180) (layer B.SilkS) hide
@@
       (net 2 /ANTCON))
   )
-  (module Monero_HW:HCPPNewordconf (layer F.Cu)
+  (module ByteRub_HW:HCPPNewordconf (layer F.Cu)
     (at 158.25 83.5)
     (fp_text reference GFX* (at 0 0) (layer F.SilkS) hide
@@
       (xy -4.544115 -10.237097) (xy -4.480005 -10.249719) (xy -4.433309 -10.242211)) (layer F.SilkS) (width 0.01))
   )
-  (module Monero_HW:HCPPNewordinst (layer F.Cu)
+  (module ByteRub_HW:HCPPNewordinst (layer F.Cu)
     (at 109 107)
     (fp_text reference GFX* (at 0 0) (layer F.SilkS) hide
@@
       (xy 4.757835 -8.636999) (xy 4.761071 -8.636709)) (layer F.SilkS) (width 0.01))
   )
-  (module Monero_HW:Fiducial_1mm_Dia_2mm_Outer (layer F.Cu)
+  (module ByteRub_HW:Fiducial_1mm_Dia_2mm_Outer (layer F.Cu)
     (at 145 55)
     (descr "Circular Fiducial, 1mm bare copper; 2mm keepout (Level A)")
@@
       (net 3 "Net-(FID1-Pad~)") (solder_mask_margin 0.5) (clearance 0.5))
   )
-  (module Monero_HW:Fiducial_1mm_Dia_2mm_Outer (layer F.Cu)
+  (module ByteRub_HW:Fiducial_1mm_Dia_2mm_Outer (layer F.Cu)
     (at 102.5 116)
     (descr "Circular Fiducial, 1mm bare copper; 2mm keepout (Level A)")
@@
       (net 4 "Net-(FID2-Pad~)") (solder_mask_margin 0.5) (clearance 0.5))
   )
-  (module Monero_HW:Fiducial_1mm_Dia_2mm_Outer (layer F.Cu)
+  (module ByteRub_HW:Fiducial_1mm_Dia_2mm_Outer (layer F.Cu)
     (at 177.5 116)
     (descr "Circular Fiducial, 1mm bare copper; 2mm keepout (Level A)")
@@
       (net 5 "Net-(FID3-Pad~)") (solder_mask_margin 0.5) (clearance 0.5))
   )
-  (module Monero_HW:MountingHole_4.3mm_M4_ISO14580_Pad (layer F.Cu)
+  (module ByteRub_HW:MountingHole_4.3mm_M4_ISO14580_Pad (layer F.Cu)
     (at 140 55)
     (descr "Mounting Hole 4.3mm, M4, ISO14580")
@@
       (net 6 GND))
   )
-  (module Monero_HW:SW_SPST_PTS645 (layer F.Cu)
+  (module ByteRub_HW:SW_SPST_PTS645 (layer F.Cu)
     (at 149.75 67.5 120)
     (descr "C&K Components SPST SMD PTS645 Series 6mm Tact Switch")
@@
     )
   )
-  (module Monero_HW:SOIC-8_3.9x4.9mm_Pitch1.27mm (layer F.Cu)
+  (module ByteRub_HW:SOIC-8_3.9x4.9mm_Pitch1.27mm (layer F.Cu)
     (at 134.5 60.5 330)
     (descr "8-Lead Plastic Small Outline (SN) - Narrow, 3.90 mm Body [SOIC] (see Microchip Packaging Specification 00000049BS.pdf)")
@@
     )
   )
-  (module Monero_HW:SOIC-8_3.9x4.9mm_Pitch1.27mm (layer F.Cu)
+  (module ByteRub_HW:SOIC-8_3.9x4.9mm_Pitch1.27mm (layer F.Cu)
     (at 145.5 60.5 210)
     (descr "8-Lead Plastic Small Outline (SN) - Narrow, 3.90 mm Body [SOIC] (see Microchip Packaging Specification 00000049BS.pdf)")
@@
     )
   )
-  (module Monero_HW:SW_SPST_K21102SP (layer F.Cu)
+  (module ByteRub_HW:SW_SPST_K21102SP (layer F.Cu)
     (at 130 68 240)
     (descr "Hro Electronics SPST SMD K2-1102SP-C4SC-04 6mm Tact Switch")
@@
     )
   )
-  (module Monero_HW:HCPPSponsors (layer B.Cu)
+  (module ByteRub_HW:HCPPSponsors (layer B.Cu)
     (at 140 88 180)
     (fp_text reference LOGO* (at 0 0 180) (layer B.SilkS) hide
