File: hardware/utilities/usbcontst/usbconntest.kicad_pcb (KiCad board)
At the start: 2 copper layers, 66 x 21 mm, 6 parts, among them J1 CONN_01X24, J3 CONN_01X24, P1 USB_C_Plug

Commit message: master
Parts:
- FID1, FID2, FID3: footprint Monero_HW:Fiducial_1mm_Dia_2mm_Outer -> ByteRub_HW:Fiducial_1mm_Dia_2mm_Outer
- J1, J3: footprint Monero_HW:Pin_Header_Straight_1x24_Pitch2.54mm -> ByteRub_HW:Pin_Header_Straight_1x24_Pitch2.54mm
- P1: footprint Monero_HW:USB_C_Plug_Molex_105444 -> ByteRub_HW:USB_C_Plug_Molex_105444
Other:
- board text added: "Copyright ©2018 The ByteRub Project"
- board text removed: "Copyright ©2018 The Monero Project"
Changed lines of the file:
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@@
     (date 2018-09-10)
     (rev 0.7)
-    (company "The Monero Project Hardware Team")
-    (comment 1 "Copyright © 2018, The Monero Project")
+    (company "The ByteRub Project Hardware Team")
+    (comment 1 "Copyright © 2018, The ByteRub Project")
     (comment 2 "Enabling testing of USB-C hardware")
     (comment 3 "Pending quality assurance testing")
@@
     (add_net "Net-(J3-Pad24)")
   )
-  (module Monero_HW:Pin_Header_Straight_1x24_Pitch2.54mm (layer F.Cu)
+  (module ByteRub_HW:Pin_Header_Straight_1x24_Pitch2.54mm (layer F.Cu)
     (at 72 89 90)
     (descr "Through hole straight pin header, 1x24, 2.54mm pitch, single row")
@@
     )
   )
-  (module Monero_HW:Pin_Header_Straight_1x24_Pitch2.54mm (layer F.Cu)
+  (module ByteRub_HW:Pin_Header_Straight_1x24_Pitch2.54mm (layer F.Cu)
     (at 72 96 90)
     (descr "Through hole straight pin header, 1x24, 2.54mm pitch, single row")
@@
       (net 26 "Net-(J3-Pad24)"))
   )
-  (module Monero_HW:USB_C_Plug_Molex_105444 (layer F.Cu)
+  (module ByteRub_HW:USB_C_Plug_Molex_105444 (layer F.Cu)
     (at 101.25 80)
     (descr "Universal Serial Bus (USB) Shielded I/O Plug, Type C, Right Angle, Surface Mount, http://www.molex.com/pdm_docs/sd/1054440001_sd.pdf")
@@
     )
   )
-  (module Monero_HW:Fiducial_1mm_Dia_2mm_Outer (layer F.Cu)
+  (module ByteRub_HW:Fiducial_1mm_Dia_2mm_Outer (layer F.Cu)
     (at 73 84)
     (descr "Circular Fiducial, 1mm bare copper; 2mm keepout (Level A)")
@@
       (net 27 "Net-(FID1-Pad~)") (solder_mask_margin 0.5) (clearance 0.5))
   )
-  (module Monero_HW:Fiducial_1mm_Dia_2mm_Outer (layer F.Cu)
+  (module ByteRub_HW:Fiducial_1mm_Dia_2mm_Outer (layer F.Cu)
     (at 128 84)
     (descr "Circular Fiducial, 1mm bare copper; 2mm keepout (Level A)")
@@
       (net 28 "Net-(FID2-Pad~)") (solder_mask_margin 0.5) (clearance 0.5))
   )
-  (module Monero_HW:Fiducial_1mm_Dia_2mm_Outer (layer F.Cu)
+  (module ByteRub_HW:Fiducial_1mm_Dia_2mm_Outer (layer F.Cu)
     (at 132 98)
     (descr "Circular Fiducial, 1mm bare copper; 2mm keepout (Level A)")
@@
     (effects (font (size 2 2) (thickness 0.3)) (justify mirror))
   )
-  (gr_text "Copyright ©2018 The Monero Project" (at 101 92.25) (layer B.SilkS)
+  (gr_text "Copyright ©2018 The ByteRub Project" (at 101 92.25) (layer B.SilkS)
     (effects (font (size 2 2) (thickness 0.3)) (justify mirror))
   )
