File: hardware/saddons/35c3re/35C3XMR.kicad_pcb (KiCad board)
At the start: 2 copper layers, 100 x 95 mm, 97 parts, among them U1 TLC555, U2 NC7SZ04L6X

Commit message: master
Parts:
- C1, C2: footprint Monero_Local:C_0805 -> ByteRub_Local:C_0805
- CR2450-A, CR2450-B: footprint Monero_Local:BatteryHolder_Keystone_3008_1x2450 -> ByteRub_Local:BatteryHolder_Keystone_3008_1x2450
- D1, D10, D11, D12, D13, D14, D15, D16, D17, D18, D19, D2, D20, D21, D22, D23, D24, D25, D26, D27, D28, D29, D3, D30, D31, D32, D33, D34, D35, D36, D37, D38, D39, D4, D40, D41, D42, D43, D44, D45, D46, D47, D48, D49, D5, D50, D51, D52, D53, D54, D55, D56, D6, D7, D8, D9: footprint Monero_Local:LED_1206 -> ByteRub_Local:LED_1206
- Dch, GND, Inv, Out, Trig, VCC: footprint Monero_Local:TestPoint_THTPad_D1.5mm_Drill0.7mm -> ByteRub_Local:TestPoint_THTPad_D1.5mm_Drill0.7mm
- FID1, FID2, FID3, FID4, FID5, FID6: footprint Monero_Local:Fiducial_1mm_Dia_2.54mm -> ByteRub_Local:Fiducial_1mm_Dia_2.54mm
- G1: footprint Monero_Local:Kastelospecsqr -> ByteRub_Local:Kastelospecsqr
- LOGO1: footprint Monero_Local:35C3Funny -> ByteRub_Local:35C3Funny
- LOGO2: value Moneroball -> ByteRubball; footprint Monero_Local:Moneroball_15mm -> ByteRub_Local:ByteRubball_15mm
- MH1, MH2, MH3, MH4: footprint Monero_Local:MountingHole_2.5mm -> ByteRub_Local:MountingHole_2.5mm
- NC, R1, R2: footprint Monero_Local:R_0805 -> ByteRub_Local:R_0805
- SAO1: footprint Monero_Local:PinHeader_2x02_P2.54mm_Vertical_SMD -> ByteRub_Local:PinHeader_2x02_P2.54mm_Vertical_SMD
- SF1, SF2, SF3, SF4, SF5: footprint Monero_Local:Solderarea -> ByteRub_Local:Solderarea
- TAB1, TAB2A, TAB2B, TAB3, TAB4, TAB5, TAB6: footprint Monero_Local:Panel_Mousetab_25mm_Single -> ByteRub_Local:Panel_Mousetab_25mm_Single
- U1: footprint Monero_Local:SOIC-8_3.9x4.9mm_P1.27mm -> ByteRub_Local:SOIC-8_3.9x4.9mm_P1.27mm
- U2: footprint Monero_Local:Fairchild_MicroPak-6_1.0x1.45mm_P0.5mm -> ByteRub_Local:Fairchild_MicroPak-6_1.0x1.45mm_P0.5mm
Other:
- board text added: "Copyright © 2018, The ByteRub Project CERN Open Hardware Licence 1.2 Astable CMOS Timer Badge 0.8.5"
- board text removed: "Copyright © 2018, The Monero Project CERN Open Hardware Licence 1.2 Astable CMOS Timer Badge 0.8.5"
