File: hardware/confbadge/defconfc/defconfc.kicad_pcb (KiCad board)
At the start: 2 copper layers, 70 x 100 mm, 39 parts, among them J1 Conn_02x03_Odd_Even, J2 Conn_02x03_Odd_Even, SW1 SW_SPST, SW2 SW_SPST, SW3 SW_SPST, SW4 SW_SPDT, U1 M24SR16-YMN6T/2, U2 M24SR16-YMN6T/2, U3 ATTINY13A-SSU

Commit message: master
Parts:
- AE1: footprint Monero_HW:NFCAntennaloop -> ByteRub_HW:NFCAntennaloop
- BT1: footprint Monero_HW:Keystone_3034_1x2032-Coincell -> ByteRub_HW:Keystone_3034_1x2032-Coincell
- FID3: footprint Monero_HW:Fiducial_1mm_Dia_2mm_Outer -> ByteRub_HW:Fiducial_1mm_Dia_2mm_Outer
- G1: footprint Monero_HW:NFCGraphicsrear -> ByteRub_HW:NFCGraphicsrear
- G2: footprint Monero_HW:Kastelospecsqrcode -> ByteRub_HW:Kastelospecsqrcode
- L2: footprint Monero_HW:Monerologokreis -> ByteRub_HW:ByteRublogokreis
- LH1, LH2: footprint Monero_HW:LanyardHole_16mm_Pad -> ByteRub_HW:LanyardHole_16mm_Pad
Other:
- board text added: "CERN licensed © The ByteRub Project 2018"
- board text added: "Designed and assembled by The ByteRub Hardware Team"
- board text removed: "CERN licensed © The Monero Project 2018"
- board text removed: "Designed and assembled by The Monero Hardware Team"
Changed lines of the file:
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@@
     (date 2018-06-22)
     (rev 1.0.0)
-    (company "The Monero Project, Hardware Team")
-    (comment 1 "Copyright © 2018, The Monero Project")
+    (company "The ByteRub Project, Hardware Team")
+    (comment 1 "Copyright © 2018, The ByteRub Project")
     (comment 2 "Fulfilling the first annual village role")
     (comment 3 "Pending quality assurance testing")
@@
       (net 2 GND))
   )
-  (module Monero_HW:LanyardHole_16mm_Pad (layer F.Cu)
+  (module ByteRub_HW:LanyardHole_16mm_Pad (layer F.Cu)
     (at 68 57)
     (descr "Lanyard Slot 16mm")
@@
       (net 2 GND))
   )
-  (module Monero_HW:LanyardHole_16mm_Pad (layer F.Cu)
+  (module ByteRub_HW:LanyardHole_16mm_Pad (layer F.Cu)
     (at 114 57)
     (descr "Lanyard Slot 16mm")
@@
       (net 2 GND))
   )
-  (module Monero_HW:Keystone_3034_1x2032-Coincell (layer B.Cu)
+  (module ByteRub_HW:Keystone_3034_1x2032-Coincell (layer B.Cu)
     (at 91 61)
     (descr "Keystone 3034 SMD battery holder for 2020, 2025 and 2032 coincell batteries. http://www.keyelco.com/product-pdf.cfm?p=798")
@@
     )
   )
-  (module Monero_HW:NFCGraphicsrear (layer B.Cu)
+  (module ByteRub_HW:NFCGraphicsrear (layer B.Cu)
     (at 91 125.75)
     (fp_text reference G1 (at 0 0) (layer B.SilkS) hide
@@
       (xy -4.73949 2.368591) (xy -4.601634 2.451835) (xy -4.455358 2.451138)) (layer B.SilkS) (width 0.01))
   )
-  (module Monero_HW:NFCAntennaloop (layer B.Cu)
+  (module ByteRub_HW:NFCAntennaloop (layer B.Cu)
     (at 91 125)
     (fp_text reference AE1 (at 0 1) (layer B.SilkS) hide
@@
       (net 14 "Net-(AE1-Pad2)"))
   )
-  (module Monero_HW:Kastelospecsqrcode (layer B.Cu)
+  (module ByteRub_HW:Kastelospecsqrcode (layer B.Cu)
     (at 104 90)
     (fp_text reference G2 (at 0 0) (layer B.SilkS) hide
@@
       (xy 2.275417 10.503958)) (layer B.SilkS) (width 0.01))
   )
-  (module Monero_HW:Monerologokreis (layer B.Cu)
+  (module ByteRub_HW:ByteRublogokreis (layer B.Cu)
     (at 82.5 84.25 180)
     (fp_text reference L2 (at 0 0 180) (layer B.SilkS) hide
@@
       (xy -0.090783 1.603289) (xy 0.156781 1.601805)) (layer B.SilkS) (width 0.01))
   )
-  (module Monero_HW:Fiducial_1mm_Dia_2mm_Outer (layer F.Cu)
+  (module ByteRub_HW:Fiducial_1mm_Dia_2mm_Outer (layer F.Cu)
     (at 120 135)
     (descr "Circular Fiducial, 1mm bare copper; 2mm keepout (Level A)")
@@
   )
   (gr_line (start 64 92) (end 85.5 92) (angle 90) (layer B.SilkS) (width 1))
-  (gr_text "CERN licensed\n© The Monero\nProject 2018" (at 86 99.5) (layer B.SilkS)
+  (gr_text "CERN licensed\n© The ByteRub\nProject 2018" (at 86 99.5) (layer B.SilkS)
     (effects (font (size 2 2) (thickness 0.5)) (justify left mirror))
   )
-  (gr_text "Designed and\nassembled by\n    The Monero\nHardware Team" (at 86 82.5) (layer B.SilkS)
+  (gr_text "Designed and\nassembled by\n    The ByteRub\nHardware Team" (at 86 82.5) (layer B.SilkS)
     (effects (font (size 2 2) (thickness 0.5)) (justify left mirror))
   )

Commit message: master ByteRub
Other:
- board text added: "BCOS|BYTERUB"
- board text removed: "BCOS|MONERO"
Changed lines of the file:
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@@
     (effects (font (size 4 4) (thickness 1)) (justify mirror))
   )
-  (gr_text BCOS|MONERO (at 91 135) (layer F.SilkS)
+  (gr_text BCOS|BYTERUB (at 91 135) (layer F.SilkS)
     (effects (font (size 4.2 4.2) (thickness 1)))
   )
